Commit message: 我的修改

File: vrx_urdf/wamv_gazebo/urdf/components/ball_shooter.xacro (robot description, xacro)
@@ -96,5 +96,5 @@
           <model_name>blue_projectile</model_name>
           <link_name>link</link_name>
-          <frame>wamv/ball_shooter_launcher_link</frame>
+          <frame>${namespace}/ball_shooter_launcher_link</frame>
           <pose>0.14 0 0 0 0 0</pose>
         </projectile>

File: vrx_urdf/wamv_gazebo/urdf/components/wamv_3d_lidar.xacro (robot description, xacro)
@@ -153,4 +153,5 @@
       <sensor type="gpu_ray" name="${name}_sensor">
         <update_rate>${update_rate}</update_rate>
+        <visualize>true</visualize>
         <ray>
           <visibility_mask>7</visibility_mask>

File: vrx_urdf/wamv_gazebo/urdf/components/wamv_imu.xacro (robot description, xacro)
@@ -3,5 +3,5 @@
   <xacro:macro name="wamv_imu" params="name:=imu x:=0.3 y:=0.5 z:=1.3 R:=0 P:=0 Y:=0 update_rate:=100">
     <link name="${namespace}/${name}_link">
-      <visual name="${name}_visual">>
+      <visual name="${name}_visual">
         <geometry>
           <box size="0.05 0.025 0.005" />
@@ -11,5 +11,5 @@
         </material>
       </visual>
-      <collision name="${name}_collision">>
+      <collision name="${name}_collision">
         <geometry>
           <box size="0.05 0.025 0.005" />

File: vrx_urdf/wamv_gazebo/urdf/thruster_layouts/wamv_gazebo_thruster_config.xacro (robot description, xacro)
@@ -5,14 +5,20 @@
     <xacro:property name="x_uu" value="72.4" />
     <xacro:property name="x_u" value="51.3" />
+    <!-- 最大转速（7.71667 m/s），用于计算最大推力大小。 -->
     <xacro:property name="max_velocity_mps" value="7.71667" />
+<!-- https://gazebosim.org/api/sim/10/classgz_1_1sim_1_1systems_1_1Thruster.html -->
     <plugin
       filename="gz-sim-thruster-system"
       name="gz::sim::systems::Thruster">
+      <!-- 指定被控制的关节，即右侧发动机的螺旋桨旋转关节。 -->
       <joint_name>${namespace}/${name}_engine_propeller_joint</joint_name>
+      <!-- 推力系数（0.004422），用于根据转速计算推力大小。 -->
       <thrust_coefficient>0.004422</thrust_coefficient>
       <fluid_density>1000</fluid_density>
+      <!-- 螺旋桨直径（0.2），用于计算推力大小。 -->
       <propeller_diameter>0.2</propeller_diameter>
+      <!-- 是否使用速度控制模式（true），默认值为false。 设为 true，表示输入指令是角速度（rad/s），而非力/扭矩。-->
       <velocity_control>true</velocity_control>
-      <!-- max total thrust / 2 -->
+      <!-- max total thrust / 2 ，用于限制最大推力大小。  -->
       <max_thrust_cmd>${((x_u + x_uu * max_velocity_mps) * max_velocity_mps)/ 2}</max_thrust_cmd>
       <namespace>${namespace}</namespace>
